File: LED_grid/LED_grid.sch (KiCad schematic (older format))
At the start: 11 parts

Commit message: Added additional led grid without controllers
Parts:
- added J1: Conn_01x13, Connector_PinHeader_2.54mm:PinHeader_1x13_P2.54mm_Vertical, symbol Connector_Generic:Conn_01x13
- gave numbers to parts that had none: 11
Connections:
- wire segments 334 -> 347
Changed lines of the file:
@@
 EESchema Schematic File Version 4
+LIBS:LED_grid-cache
 EELAYER 26 0
 EELAYER END
@@
 Wire Wire Line
 	7750 2750 8250 2750
-Text HLabel 9600 1950 2    50   Input ~ 0
-DIN
-Text HLabel 9600 2050 2    50   Input ~ 0
-DCLK
 Entry Wire Line
 	9400 1850 9500 1950
@@
 	8800 5600 8950 5600
 $Comp
-L Transistor_BJT:BD135 Q?
+L Transistor_BJT:BD135 Q2
 U 1 1 5DF57628
 P 1950 6500
-F 0 "Q?" V 2141 6546 50  0000 C TNN
+F 0 "Q2" V 2141 6546 50  0000 C TNN
 F 1 "FMMT620CT-ND" V 2141 6455 50  0001 L TNN
 F 2 "Package_TO_SOT_SMD:SOT-23_Handsoldering" H 2150 6425 50  0001 L CIN
@@
 $EndComp
 $Comp
-L Transistor_BJT:BD135 Q?
+L Transistor_BJT:BD135 Q1
 U 1 1 5DF9866A
 P 1300 6500
-F 0 "Q?" V 1491 6546 50  0000 C TNN
+F 0 "Q1" V 1491 6546 50  0000 C TNN
 F 1 "FMMT620CT-ND" V 1491 6455 50  0001 L TNN
 F 2 "Package_TO_SOT_SMD:SOT-23_Handsoldering" H 1500 6425 50  0001 L CIN
@@
 $EndComp
 $Comp
-L Transistor_BJT:BD135 Q?
+L Transistor_BJT:BD135 Q4
 U 1 1 5DFD9643
 P 3250 6500
-F 0 "Q?" V 3441 6546 50  0000 C TNN
+F 0 "Q4" V 3441 6546 50  0000 C TNN
 F 1 "FMMT620CT-ND" V 3441 6455 50  0001 L TNN
 F 2 "Package_TO_SOT_SMD:SOT-23_Handsoldering" H 3450 6425 50  0001 L CIN
@@
 $EndComp
 $Comp
-L Transistor_BJT:BD135 Q?
+L Transistor_BJT:BD135 Q3
 U 1 1 5E01A615
 P 2600 6500
-F 0 "Q?" V 2791 6546 50  0000 C TNN
+F 0 "Q3" V 2791 6546 50  0000 C TNN
 F 1 "FMMT620CT-ND" V 2791 6455 50  0001 L TNN
 F 2 "Package_TO_SOT_SMD:SOT-23_Handsoldering" H 2800 6425 50  0001 L CIN
@@
 $EndComp
 $Comp
-L Transistor_BJT:BD135 Q?
+L Transistor_BJT:BD135 Q11
 U 1 1 5E05B5E4
 P 3900 7450
-F 0 "Q?" V 4091 7496 50  0000 C TNN
+F 0 "Q11" V 4091 7496 50  0000 C TNN
 F 1 "FMMT620CT-ND" V 4091 7405 50  0001 L TNN
 F 2 "Package_TO_SOT_SMD:SOT-23_Handsoldering" H 4100 7375 50  0001 L CIN
@@
 $EndComp
 $Comp
-L Transistor_BJT:BD135 Q?
+L Transistor_BJT:BD135 Q6
 U 1 1 5E09C5B6
 P 4550 6500
-F 0 "Q?" V 4741 6546 50  0000 C TNN
+F 0 "Q6" V 4741 6546 50  0000 C TNN
 F 1 "FMMT620CT-ND" V 4741 6455 50  0001 L TNN
 F 2 "Package_TO_SOT_SMD:SOT-23_Handsoldering" H 4750 6425 50  0001 L CIN
@@
 $EndComp
 $Comp
-L Transistor_BJT:BD135 Q?
+L Transistor_BJT:BD135 Q5
 U 1 1 5E0DD589
 P 3900 6500
-F 0 "Q?" V 4091 6546 50  0000 C TNN
+F 0 "Q5" V 4091 6546 50  0000 C TNN
 F 1 "FMMT620CT-ND" V 4091 6455 50  0001 L TNN
 F 2 "Package_TO_SOT_SMD:SOT-23_Handsoldering" H 4100 6425 50  0001 L CIN
@@
 $EndComp
 $Comp
-L Transistor_BJT:BD135 Q?
+L Transistor_BJT:BD135 Q7
 U 1 1 5E4ED363
 P 1300 7450
-F 0 "Q?" V 1491 7496 50  0000 C TNN
+F 0 "Q7" V 1491 7496 50  0000 C TNN
 F 1 "FMMT620CT-ND" V 1491 7405 50  0001 L TNN
 F 2 "Package_TO_SOT_SMD:SOT-23_Handsoldering" H 1500 7375 50  0001 L CIN
@@
 $EndComp
 $Comp
-L Transistor_BJT:BD135 Q?
+L Transistor_BJT:BD135 Q10
 U 1 1 5E4ED36A
 P 3250 7450
-F 0 "Q?" V 3441 7496 50  0000 C TNN
+F 0 "Q10" V 3441 7496 50  0000 C TNN
 F 1 "FMMT620CT-ND" V 3441 7405 50  0001 L TNN
 F 2 "Package_TO_SOT_SMD:SOT-23_Handsoldering" H 3450 7375 50  0001 L CIN
@@
 $EndComp
 $Comp
-L Transistor_BJT:BD135 Q?
+L Transistor_BJT:BD135 Q9
 U 1 1 5E4ED371
 P 2600 7450
-F 0 "Q?" V 2791 7496 50  0000 C TNN
+F 0 "Q9" V 2791 7496 50  0000 C TNN
 F 1 "FMMT620CT-ND" V 2791 7405 50  0001 L TNN
 F 2 "Package_TO_SOT_SMD:SOT-23_Handsoldering" H 2800 7375 50  0001 L CIN
@@
 $EndComp
 $Comp
-L Transistor_BJT:BD135 Q?
+L Transistor_BJT:BD135 Q8
 U 1 1 5E4ED378
 P 1950 7450
-F 0 "Q?" V 2141 7496 50  0000 C TNN
+F 0 "Q8" V 2141 7496 50  0000 C TNN
 F 1 "FMMT620CT-ND" V 2141 7405 50  0001 L TNN
 F 2 "Package_TO_SOT_SMD:SOT-23_Handsoldering" H 2150 7375 50  0001 L CIN
@@
 $EndComp
 $Comp
-L power:+5V #PWR?
+L power:+5V #PWR01
 U 1 1 5E56F3AB
 P 1200 6700
-F 0 "#PWR?" H 1200 6550 50  0001 C CNN
+F 0 "#PWR01" H 1200 6550 50  0001 C CNN
 F 1 "+5V" V 1215 6828 50  0000 L CNN
 F 2 "" H 1200 6700 50  0001 C CNN
@@
 $EndComp
 $Comp
-L power:+5V #PWR?
+L power:+5V #PWR02
 U 1 1 5E5B0420
 P 1850 6700
-F 0 "#PWR?" H 1850 6550 50  0001 C CNN
+F 0 "#PWR02" H 1850 6550 50  0001 C CNN
 F 1 "+5V" V 1865 6828 50  0000 L CNN
 F 2 "" H 1850 6700 50  0001 C CNN
@@
 $EndComp
 $Comp
-L power:+5V #PWR?
+L power:+5V #PWR03
 U 1 1 5E5F0726
 P 2500 6700
-F 0 "#PWR?" H 2500 6550 50  0001 C CNN
+F 0 "#PWR03" H 2500 6550 50  0001 C CNN
 F 1 "+5V" V 2515 6828 50  0000 L CNN
 F 2 "" H 2500 6700 50  0001 C CNN
@@
 $EndComp
 $Comp
-L power:+5V #PWR?
+L power:+5V #PWR04
 U 1 1 5E630A47
 P 3150 6700
-F 0 "#PWR?" H 3150 6550 50  0001 C CNN
+F 0 "#PWR04" H 3150 6550 50  0001 C CNN
 F 1 "+5V" V 3165 6828 50  0000 L CNN
 F 2 "" H 3150 6700 50  0001 C CNN
@@
 $EndComp
 $Comp
-L power:+5V #PWR?
+L power:+5V #PWR05
 U 1 1 5E670D68
 P 3800 6700
-F 0 "#PWR?" H 3800 6550 50  0001 C CNN
+F 0 "#PWR05" H 3800 6550 50  0001 C CNN
 F 1 "+5V" V 3815 6828 50  0000 L CNN
 F 2 "" H 3800 6700 50  0001 C CNN
@@
 $EndComp
 $Comp
-L power:+5V #PWR?
+L power:+5V #PWR06
 U 1 1 5E6B1089
 P 4450 6700
-F 0 "#PWR?" H 4450 6550 50  0001 C CNN
+F 0 "#PWR06" H 4450 6550 50  0001 C CNN
 F 1 "+5V" V 4465 6828 50  0000 L CNN
 F 2 "" H 4450 6700 50  0001 C CNN
@@
 $EndComp
 $Comp
-L power:+5V #PWR?
+L power:+5V #PWR07
 U 1 1 5E7316CA
 P 1200 7650
-F 0 "#PWR?" H 1200 7500 50  0001 C CNN
+F 0 "#PWR07" H 1200 7500 50  0001 C CNN
 F 1 "+5V" V 1215 7778 50  0000 L CNN
 F 2 "" H 1200 7650 50  0001 C CNN
@@
 $EndComp
 $Comp
-L power:+5V #PWR?
+L power:+5V #PWR08
 U 1 1 5E7719EB
 P 1850 7650
-F 0 "#PWR?" H 1850 7500 50  0001 C CNN
+F 0 "#PWR08" H 1850 7500 50  0001 C CNN
 F 1 "+5V" V 1865 7778 50  0000 L CNN
 F 2 "" H 1850 7650 50  0001 C CNN
@@
 $EndComp
 $Comp
-L power:+5V #PWR?
+L power:+5V #PWR09
 U 1 1 5E7B1D0C
 P 2500 7650
-F 0 "#PWR?" H 2500 7500 50  0001 C CNN
+F 0 "#PWR09" H 2500 7500 50  0001 C CNN
 F 1 "+5V" V 2515 7778 50  0000 L CNN
 F 2 "" H 2500 7650 50  0001 C CNN
@@
 $EndComp
 $Comp
-L power:+5V #PWR?
+L power:+5V #PWR010
 U 1 1 5E7F202D
 P 3150 7650
-F 0 "#PWR?" H 3150 7500 50  0001 C CNN
+F 0 "#PWR010" H 3150 7500 50  0001 C CNN
 F 1 "+5V" V 3165 7778 50  0000 L CNN
 F 2 "" H 3150 7650 50  0001 C CNN
@@
 $EndComp
 $Comp
-L power:+5V #PWR?
+L power:+5V #PWR011
 U 1 1 5E83234E
 P 3800 7650
-F 0 "#PWR?" H 3800 7500 50  0001 C CNN
+F 0 "#PWR011" H 3800 7500 50  0001 C CNN
 F 1 "+5V" V 3815 7778 50  0000 L CNN
 F 2 "" H 3800 7650 50  0001 C CNN
@@
 	0    -1   -1   0
 $EndComp
-Text HLabel 1500 6500 1    50   Input ~ 0
-ROW0
-Text HLabel 2150 6500 1    50   Input ~ 0
-ROW1
-Text HLabel 2800 6500 1    50   Input ~ 0
-ROW2
-Text HLabel 3450 6500 1    50   Input ~ 0
-ROW3
-Text HLabel 4100 6500 1    50   Input ~ 0
-ROW4
-Text HLabel 4750 6500 1    50   Input ~ 0
-ROW5
-Text HLabel 1500 7450 1    50   Input ~ 0
-ROW6
-Text HLabel 2150 7450 1    50   Input ~ 0
-ROW7
-Text HLabel 2800 7450 1    50   Input ~ 0
-ROW8
-Text HLabel 3450 7450 1    50   Input ~ 0
-ROW9
-Text HLabel 4100 7450 1    50   Input ~ 0
-ROW10
 Wire Bus Line
 	700  7100 700  6100
@@
 Wire Wire Line
 	4450 6300 4450 6200
+$Comp
+L Connector_Generic:Conn_01x13 J1
+U 1 1 5C082F8E
+P 10700 3250
+F 0 "J1" H 10780 3292 50  0000 L CNN
+F 1 "Conn_01x13" H 10780 3201 50  0000 L CNN
+F 2 "Connector_PinHeader_2.54mm:PinHeader_1x13_P2.54mm_Vertical" H 10700 3250 50  0001 C CNN
+F 3 "~" H 10700 3250 50  0001 C CNN
+	1    10700 3250
+	1    0    0    -1
+$EndComp
+Text Label 10450 3750 2    50   ~ 0
+DIN
+Text Label 10450 3850 2    50   ~ 0
+DCLK
+Wire Wire Line
+	10450 3750 10500 3750
+Wire Wire Line
+	10450 3850 10500 3850
+Text Label 4100 6500 0    50   ~ 0
+ROW4
+Text Label 3450 6500 0    50   ~ 0
+ROW3
+Text Label 2800 6500 0    50   ~ 0
+ROW2
+Text Label 2150 6500 0    50   ~ 0
+ROW1
+Text Label 1500 6500 0    50   ~ 0
+ROW0
+Text Label 4750 6500 0    50   ~ 0
+ROW5
+Text Label 1500 7450 0    50   ~ 0
+ROW6
+Text Label 2150 7450 0    50   ~ 0
+ROW7
+Text Label 2800 7450 0    50   ~ 0
+ROW8
+Text Label 3450 7450 0    50   ~ 0
+ROW9
+Text Label 4100 7450 0    50   ~ 0
+ROW10
+Text Label 10450 2650 2    50   ~ 0
+ROW0
+Text Label 10450 2750 2    50   ~ 0
+ROW1
+Text Label 10450 2850 2    50   ~ 0
+ROW2
+Text Label 10450 2950 2    50   ~ 0
+ROW3
+Text Label 10450 3050 2    50   ~ 0
+ROW4
+Text Label 10450 3150 2    50   ~ 0
+ROW5
+Text Label 10450 3250 2    50   ~ 0
+ROW6
+Text Label 10450 3350 2    50   ~ 0
+ROW7
+Text Label 10450 3450 2    50   ~ 0
+ROW8
+Text Label 10450 3550 2    50   ~ 0
+ROW9
+Text Label 10450 3650 2    50   ~ 0
+ROW10
+Wire Wire Line
+	10500 2650 10450 2650
+Wire Wire Line
+	10450 2750 10500 2750
+Wire Wire Line
+	10450 2850 10500 2850
+Wire Wire Line
+	10450 2950 10500 2950
+Wire Wire Line
+	10450 3050 10500 3050
+Wire Wire Line
+	10450 3150 10500 3150
+Wire Wire Line
+	10450 3250 10500 3250
+Wire Wire Line
+	10450 3350 10500 3350
+Wire Wire Line
+	10450 3450 10500 3450
+Wire Wire Line
+	10450 3550 10500 3550
+Wire Wire Line
+	10450 3650 10500 3650
 Wire Bus Line
 	9400 600  9400 2650
