File: LED_grid/PWM_controller.sch (KiCad schematic (older format))
At the start: 7 parts, among them Q0 2N3904, Q1 2N3904, Q2 2N3904

Commit message: Added additional led grid without controllers
Parts:
- removed R0: 150, symbol Device:R
- removed R1, R2: 100, symbol Device:R
- added R?: 100, Resistor_THT:R_Axial_DIN0207_L6.3mm_D2.5mm_P10.16mm_Horizontal, symbol Device:R_US
- added R? (x2): 150, Resistor_THT:R_Axial_DIN0207_L6.3mm_D2.5mm_P10.16mm_Horizontal, symbol Device:R_US
- added R?: 10k, symbol Device:R_US
- added RN?: R_Pack03_SIP_10k, Resistor_THT:R_Array_SIP6, symbol Device:R_Pack03_SIP
- renumbered Q0 to Q?, Q1 to Q?, Q2 to Q?
Connections:
- net labels added: B_RES_OUT, G_RES_OUT, R_RES_OUT
- wire segments 18 -> 9
Other:
- moved on the sheet: Q?, U?

Commit message: Added 3 updated designs and partslist for revision 1 and 2 of the led grid
Parts:
- removed Q? (x3): 2N3904, Package_TO_SOT_SMD:SOT-23_Handsoldering, symbol Transistor_BJT:2N3904
- removed R?: 10k, symbol Device:R_US
- added Q1, Q2, Q3: 2N3904_SOT-23, Package_TO_SOT_SMD:SOT-23_Handsoldering, symbol Transistor_BJT:2N3904_SOT-23
- gave numbers to parts that had none: 5
Connections:
- net labels added: Vcc
- net labels removed: +5V
