File: LED_grid_controllers/LED_grid_controllers.sch (KiCad schematic (older format))
At the start: 0 parts

Commit message: Added 3 updated designs and partslist for revision 1 and 2 of the led grid
Parts:
- added J1, J3: Conn_01x24, Connector_PinSocket_2.54mm:PinSocket_1x24_P2.54mm_Vertical, symbol Connector_Generic:Conn_01x24
- added J2: Conn_01x05, Connector_PinHeader_2.54mm:PinHeader_1x05_P2.54mm_Vertical, symbol Connector_Generic:Conn_01x05
Connections:
- net labels added: +5V, B0, B1, B10, B11, B12, B13, B14, B15, B2, B3, B4, B5, B6, B7, B8, B9, DCLK, DIN, DOUT, DOUT11, DOUT3, DOUT7, G0, G1, G10, G11, G12, G13, G14, G15, G2, G3, G4, G5, G6, G7, G8, G9, GND, R0, R1, R10, R11, R12, R13, R14, R15, R2, R3, R4, R5, R6, R7, R8, R9, Vcc
- wire segments 0 -> 177
