File: LED_grid_no_controllers/LED_grid_no_controllers.sch (KiCad schematic (older format))
At the start: 14 parts

Commit message: Added extra columns to grid along with 5V pin to connectors
Parts:
- removed J?: Conn_02x22_Odd_Even, symbol Connector_Generic:Conn_02x22_Odd_Even
- added J1: Conn_01x12, symbol Connector_Generic:Conn_01x12
- added J2: Conn_02x24_Counter_Clockwise, symbol Connector_Generic:Conn_02x24_Counter_Clockwise
- gave numbers to parts that had none: 13
Connections:
- net labels added: B11, B12, B13, B14, B15, G11, G12, G13, G14, G15, R11, R12, R13, R14, R15
- wire segments 220 -> 306
Other:
- moved on the sheet: Q10, Q11, Q2, Q3, Q4, Q5, Q6, Q7, Q8, Q9, RN1, RN2

Commit message: Added 3 updated designs and partslist for revision 1 and 2 of the led grid
Parts:
- removed J2: Conn_02x24_Counter_Clockwise, symbol Connector_Generic:Conn_02x24_Counter_Clockwise
- removed Q1, Q10, Q11, Q2, Q3, Q4, Q5, Q6, Q7, Q8, Q9: DNBT8105-7, Package_TO_SOT_THT:TO-39-3, symbol Transistor_BJT:BC141
- removed RN2: R_Pack07_SIP_10k, Resistor_THT:R_Array_SIP14, symbol Device:R_Pack07_SIP
- added J2, J3: Conn_01x24, Connector_PinHeader_2.54mm:PinHeader_1x24_P2.54mm_Vertical, symbol Connector_Generic:Conn_01x24
- added Q1, Q10, Q11, Q2, Q3, Q4, Q5, Q6, Q7, Q8, Q9: DNBT8105, Package_TO_SOT_SMD:SOT-23_Handsoldering, symbol Transistor_BJT:DNBT8105
- added RN2: R_Pack04_SIP_10k, Resistor_THT:R_Array_SIP8, symbol Device:R_Pack04_SIP
- added RN3: R_Pack03_SIP_10k, Resistor_THT:R_Array_SIP6, symbol Device:R_Pack03_SIP
- J1: footprint (none) -> Connector_PinHeader_2.54mm:PinHeader_1x12_P2.54mm_Vertical
